Commit message: Adding Nozzle Carriage

File: src/football_gumming_sim/urdf/football_gumming.urdf.xacro (robot description, xacro)
@@ -130,5 +130,5 @@
   </link>
   <joint name="rail_mount" type="fixed">
-    <parent link="base_link"/><child link="nozzle_rail"/><origin xyz="0 0 0.675"/>
+    <parent link="base_link"/><child link="nozzle_rail"/><origin xyz="0 0.055 0.675"/>
   </joint>
   <link name="z_carriage">
@@ -136,4 +136,9 @@
     <visual><geometry><box size="0.05 0.05 0.08"/></geometry><material name="rail_silver"/></visual>
     <collision><geometry><box size="0.05 0.05 0.08"/></geometry></collision>
+    <visual name="front_plate"><origin xyz="0 -0.028 0" rpy="0 0 0"/><geometry><box size="0.056 0.006 0.07"/></geometry><material name="motor_dark"/></visual>
+    <visual name="plate_bolt_-22_-28"><origin xyz="-0.022 -0.0315 -0.028" rpy="1.5708 0 0"/><geometry><cylinder radius="0.0025" length="0.003"/></geometry><material name="rail_silver"/></visual>
+    <visual name="plate_bolt_-22_28"><origin xyz="-0.022 -0.0315 0.028" rpy="1.5708 0 0"/><geometry><cylinder radius="0.0025" length="0.003"/></geometry><material name="rail_silver"/></visual>
+    <visual name="plate_bolt_22_-28"><origin xyz="0.022 -0.0315 -0.028" rpy="1.5708 0 0"/><geometry><cylinder radius="0.0025" length="0.003"/></geometry><material name="rail_silver"/></visual>
+    <visual name="plate_bolt_22_28"><origin xyz="0.022 -0.0315 0.028" rpy="1.5708 0 0"/><geometry><cylinder radius="0.0025" length="0.003"/></geometry><material name="rail_silver"/></visual>
   </link>
   <joint name="z_axis_joint" type="prismatic">
@@ -146,15 +151,21 @@
   <link name="nozzle_body">
     <inertial><mass value="0.5"/><inertia ixx="0.002604" ixy="0" ixz="0" iyy="0.002604" iyz="0" izz="0.000408"/></inertial>
-    <visual name="body"><origin xyz="0 0 0" rpy="0 0 0"/><geometry><box size="0.035 0.035 0.12"/></geometry><material name="nozzle_orange"/></visual>
-    <visual name="tip_cone"><origin xyz="0 0 -0.0675" rpy="0 0 0"/><geometry><cylinder radius="0.006" length="0.015"/></geometry><material name="rail_silver"/></visual>
-    <visual name="needle"><origin xyz="0 0 -0.08" rpy="0 0 0"/><geometry><cylinder radius="0.002" length="0.01"/></geometry><material name="rubber_black"/></visual>
-    <visual name="cartridge"><origin xyz="0.0325 0 0.03" rpy="0 0 0"/><geometry><cylinder radius="0.011" length="0.1"/></geometry><material name="glue_amber"/></visual>
-    <visual name="cartridge_cap"><origin xyz="0.0325 0 0.085" rpy="0 0 0"/><geometry><cylinder radius="0.013" length="0.01"/></geometry><material name="motor_dark"/></visual>
-    <visual name="air_line"><origin xyz="0.0325 0 0.115" rpy="0 0 0"/><geometry><cylinder radius="0.003" length="0.05"/></geometry><material name="rubber_black"/></visual>
-    <visual name="glue_tube"><origin xyz="0.025 0 -0.015" rpy="0 1.5708 0"/><geometry><cylinder radius="0.003" length="0.0175"/></geometry><material name="glue_amber"/></visual>
-    <visual name="valve"><origin xyz="0 0 0.05" rpy="0 0 0"/><geometry><box size="0.045 0.045 0.02"/></geometry><material name="motor_dark"/></visual>
+    <visual name="needle_16G"><origin xyz="0 0 -0.076" rpy="0 0 0"/><geometry><cylinder radius="0.00083" length="0.018"/></geometry><material name="rail_silver"/></visual>
+    <visual name="tip_taper"><origin xyz="0 0 -0.065" rpy="0 0 0"/><geometry><cylinder radius="0.0018" length="0.004"/></geometry><material name="nozzle_orange"/></visual>
+    <visual name="tip_taper2"><origin xyz="0 0 -0.0605" rpy="0 0 0"/><geometry><cylinder radius="0.0032" length="0.005"/></geometry><material name="nozzle_orange"/></visual>
+    <visual name="luer_hub"><origin xyz="0 0 -0.053" rpy="0 0 0"/><geometry><cylinder radius="0.0045" length="0.01"/></geometry><material name="nozzle_orange"/></visual>
+    <visual name="luer_lock_collar"><origin xyz="0 0 -0.044" rpy="0 0 0"/><geometry><cylinder radius="0.0065" length="0.008"/></geometry><material name="rail_silver"/></visual>
+    <visual name="barrel_10cc"><origin xyz="0 0 0.005" rpy="0 0 0"/><geometry><cylinder radius="0.0082" length="0.09"/></geometry><material name="glue_amber"/></visual>
+    <visual name="barrel_flange"><origin xyz="0 0 0.051" rpy="0 0 0"/><geometry><cylinder radius="0.0115" length="0.002"/></geometry><material name="motor_dark"/></visual>
+    <visual name="clamp_collar"><origin xyz="0 0 0.044" rpy="0 0 0"/><geometry><cylinder radius="0.013" length="0.012"/></geometry><material name="motor_dark"/></visual>
+    <visual name="piston_cap"><origin xyz="0 0 0.063" rpy="0 0 0"/><geometry><cylinder radius="0.0095" length="0.022"/></geometry><material name="motor_dark"/></visual>
+    <visual name="air_fitting"><origin xyz="0 0 0.078" rpy="0 0 0"/><geometry><cylinder radius="0.003" length="0.008"/></geometry><material name="rail_silver"/></visual>
+    <visual name="air_hose"><origin xyz="0 0 0.086" rpy="0 0 0"/><geometry><cylinder radius="0.002" length="0.008"/></geometry><material name="rubber_black"/></visual>
+    <visual name="holder_arm"><origin xyz="0 0.0275 0.044" rpy="0 0 0"/><geometry><box size="0.026 0.055 0.012"/></geometry><material name="motor_dark"/></visual>
+    <visual name="holder_brace"><origin xyz="0 0.0275 0.065" rpy="0 0 0"/><geometry><box size="0.014 0.055 0.008"/></geometry><material name="motor_dark"/></visual>
+    <visual name="air_hose_out"><origin xyz="0.04 0 0.09" rpy="0 1.5708 0"/><geometry><cylinder radius="0.002" length="0.08"/></geometry><material name="rubber_black"/></visual>
   </link>
   <joint name="nozzle_mount" type="fixed">
-    <parent link="z_carriage"/><child link="nozzle_body"/><origin xyz="0 0 -0.09"/>
+    <parent link="z_carriage"/><child link="nozzle_body"/><origin xyz="0 -0.055 -0.09"/>
   </joint>
   <link name="pivot_pillar">
