Commit message: FIx the nozzle up/down movement

File: src/football_gumming_sim/urdf/football_gumming.urdf.xacro (robot description, xacro)
@@ -328,7 +328,7 @@
     <parent link="nozzle_rail"/><child link="z_carriage"/>
     <origin xyz="0 -0.033 0.075"/>
-    <axis xyz="0 0 0.5"/>
-    <limit lower="-0.1000" upper="0.0500" effort="60" velocity="0.0750"/>
-    <dynamics damping="4.0" friction="0.2"/>
+    <axis xyz="0 0 1"/>
+    <limit lower="-0.1000" upper="0.0500" effort="1000" velocity="10"/>
+    <dynamics damping="0.5" friction="0.0"/>
   </joint>
   <link name="nozzle_body">
@@ -389,5 +389,5 @@
     <parent link="base_link"/><child link="tilt_link"/>
     <origin xyz="0 0 0.4"/>
-    <axis xyz="0 0.5 0"/>
+    <axis xyz="0 1 0"/>
     <limit lower="-0.9" upper="0.9" effort="200" velocity="1.0"/>
     <dynamics damping="2.0" friction="0.1"/>
@@ -403,5 +403,5 @@
     <parent link="tilt_link"/><child link="left_cup"/>
     <origin xyz="-0.125 0 0"/>
-    <axis xyz="0.5 0 0"/>
+    <axis xyz="1 0 0"/>
     <limit lower="-12.6" upper="12.6" effort="50" velocity="3.0"/>
     <dynamics damping="1.0" friction="0.05"/>
@@ -417,5 +417,5 @@
     <parent link="tilt_link"/><child link="right_cup"/>
     <origin xyz="0.125 0 0"/>
-    <axis xyz="0.5 0 0"/>
+    <axis xyz="1 0 0"/>
     <limit lower="-12.6" upper="12.6" effort="50" velocity="3.0"/>
     <dynamics damping="1.0" friction="0.05"/>
@@ -699,5 +699,5 @@
   <joint name="reclamp_joint" type="revolute">
     <parent link="left_cup"/><child link="football"/><origin xyz="0.125 0 0"/>
-    <axis xyz="0 -0.0373375 0.498604"/>
+    <axis xyz="0.000000 -0.074675 0.997208"/>
     <limit lower="0" upper="1.4021" effort="50" velocity="0.8"/>
     <dynamics damping="1.0" friction="0.05"/>
@@ -717,3 +717,5 @@
     </plugin>
   </gazebo>
+  <gazebo reference="z_carriage"><gravity>false</gravity></gazebo>
+  <gazebo reference="nozzle_body"><gravity>false</gravity></gazebo>
 </robot>

Commit message: Fixing Seam count for Balls

File: src/football_gumming_sim/urdf/football_gumming.urdf.xacro (robot description, xacro)
@@ -175,16 +175,15 @@
     <visual name="door_hinge_0.0"><origin xyz="0.69 -0.015 0.4" rpy="0 0 0"/><geometry><cylinder radius="0.006" length="0.045"/></geometry><material name="rail_silver"/></visual>
     <visual name="door_hinge_-0.3"><origin xyz="0.69 -0.015 0.25" rpy="0 0 0"/><geometry><cylinder radius="0.006" length="0.045"/></geometry><material name="rail_silver"/></visual>
-    <visual name="strip_base"><origin xyz="0.515 -0.03 0.606" rpy="0 0 0"/><geometry><box size="0.35 0.07 0.015"/></geometry><material name="enclosure_grey"/></visual>
-    <visual name="ctrl_strip"><origin xyz="0.515 -0.045 0.6175" rpy="0.45 0 0"/><geometry><box size="0.35 0.085 0.01"/></geometry><material name="motor_dark"/></visual>
-    <visual name="estop_yellow_ring"><origin xyz="0.625 -0.04848 0.624705" rpy="0.45 0 0"/><geometry><cylinder radius="0.035" length="0.006"/></geometry><material name="safety_yellow"/></visual>
-    <visual name="estop_button"><origin xyz="0.625 -0.0537 0.63551" rpy="0.45 0 0"/><geometry><cylinder radius="0.0225" length="0.015"/></geometry><material name="red_btn"/></visual>
-    <visual name="btn_start"><origin xyz="0.405 -0.04935 0.626505" rpy="0.45 0 0"/><geometry><cylinder radius="0.013" length="0.01"/></geometry><material name="green_led"/></visual>
-    <visual name="btn_stop"><origin xyz="0.445 -0.04935 0.626505" rpy="0.45 0 0"/><geometry><cylinder radius="0.013" length="0.01"/></geometry><material name="red_btn"/></visual>
-    <visual name="btn_reset"><origin xyz="0.485 -0.04935 0.626505" rpy="0.45 0 0"/><geometry><cylinder radius="0.013" length="0.01"/></geometry><material name="cabinet_blue"/></visual>
-    <visual name="key_switch"><origin xyz="0.545 -0.04935 0.626505" rpy="0.45 0 0"/><geometry><cylinder radius="0.015" length="0.0125"/></geometry><material name="rubber_black"/></visual>
-    <visual name="beacon_base"><origin xyz="0.38 0.085 0.615" rpy="0 0 0"/><geometry><cylinder radius="0.01" length="0.03"/></geometry><material name="motor_dark"/></visual>
-    <visual name="beacon_light_0"><origin xyz="0.38 0.085 0.6425" rpy="0 0 0"/><geometry><cylinder radius="0.014" length="0.025"/></geometry><material name="red_btn"/></visual>
-    <visual name="beacon_light_1"><origin xyz="0.38 0.085 0.6675" rpy="0 0 0"/><geometry><cylinder radius="0.014" length="0.025"/></geometry><material name="nozzle_orange"/></visual>
-    <visual name="beacon_light_2"><origin xyz="0.38 0.085 0.6925" rpy="0 0 0"/><geometry><cylinder radius="0.014" length="0.025"/></geometry><material name="green_led"/></visual>
+    <visual name="ctrl_deck"><origin xyz="0.515 0.035 0.605" rpy="0 0 0"/><geometry><box size="0.35 0.1 0.01"/></geometry><material name="motor_dark"/></visual>
+    <visual name="estop_yellow_ring"><origin xyz="0.625 0.035 0.613" rpy="0 0 0"/><geometry><cylinder radius="0.035" length="0.006"/></geometry><material name="safety_yellow"/></visual>
+    <visual name="estop_button"><origin xyz="0.625 0.035 0.6235" rpy="0 0 0"/><geometry><cylinder radius="0.0225" length="0.015"/></geometry><material name="red_btn"/></visual>
+    <visual name="btn_start"><origin xyz="0.405 0.035 0.615" rpy="0 0 0"/><geometry><cylinder radius="0.013" length="0.01"/></geometry><material name="green_led"/></visual>
+    <visual name="btn_stop"><origin xyz="0.445 0.035 0.615" rpy="0 0 0"/><geometry><cylinder radius="0.013" length="0.01"/></geometry><material name="red_btn"/></visual>
+    <visual name="btn_reset"><origin xyz="0.485 0.035 0.615" rpy="0 0 0"/><geometry><cylinder radius="0.013" length="0.01"/></geometry><material name="cabinet_blue"/></visual>
+    <visual name="key_switch"><origin xyz="0.545 0.035 0.61625" rpy="0 0 0"/><geometry><cylinder radius="0.015" length="0.0125"/></geometry><material name="rubber_black"/></visual>
+    <visual name="beacon_base"><origin xyz="0.38 0.125 0.615" rpy="0 0 0"/><geometry><cylinder radius="0.01" length="0.03"/></geometry><material name="motor_dark"/></visual>
+    <visual name="beacon_light_0"><origin xyz="0.38 0.125 0.6425" rpy="0 0 0"/><geometry><cylinder radius="0.014" length="0.025"/></geometry><material name="red_btn"/></visual>
+    <visual name="beacon_light_1"><origin xyz="0.38 0.125 0.6675" rpy="0 0 0"/><geometry><cylinder radius="0.014" length="0.025"/></geometry><material name="nozzle_orange"/></visual>
+    <visual name="beacon_light_2"><origin xyz="0.38 0.125 0.6925" rpy="0 0 0"/><geometry><cylinder radius="0.014" length="0.025"/></geometry><material name="green_led"/></visual>
     <visual name="drip_tray_floor"><origin xyz="0 0.025 0.1625" rpy="0 0 0"/><geometry><box size="0.25 0.2 0.005"/></geometry><material name="stainless"/></visual>
     <visual name="drip_tray_front"><origin xyz="0 -0.0725 0.175" rpy="0 0 0"/><geometry><box size="0.25 0.005 0.025"/></geometry><material name="stainless"/></visual>
